File: qlexternal512kram_MIX.kicad_pcb (KiCad board)
At the start: 2 copper layers, 97.8 x 35.6 mm, 13 parts, among them J1 QL_SLOT_DIN41612_CARD, J2 QL_SLOT_DIN41612_CARD, U1 HM628512BLFP-7, U2 GAL16V8B-25QP, U3 LM1117-5.0

Commit message: Revision 0.01
Parts:
- added kibuzzard-660FAAE3: G***, kibuzzard-660FAAE3, F.Cu at (169.6, 77.6)
- moved J1 0.05 mm to (181.1, 57.8)
Routing:
- net GND: track 278.1 -> 0.00 mm
- net VCC: track 98.2 -> 91.6 mm
- net /DTACK: track 74.4 -> 78.1 mm, vias 1 -> 3
- net /A1: track 54.6 -> 57.0 mm
- net +9V: track 48.4 -> 50.7 mm
- net /D5: track 100.1 -> 102.2 mm
- net /AS: track 65.1 -> 66.5 mm, vias 1 -> 3
- net /DSMC: track 120.7 -> 122.1 mm
- net /A18: track 101.4 -> 102.4 mm
- net /A16: track 82.2 -> 82.8 mm
- net /A15: track 77.4 -> 77.1 mm, vias 0 -> 2
- net /A3: track 59.8 -> 59.6 mm, vias 0 -> 2
- net /A17: vias 1 -> 2
- net /A13: track 48.8 -> 48.7 mm, vias 0 -> 1
- net /A2: vias 0 -> 2
- added copper zone on B.Cu, net (none)
- removed copper zone on F.Cu, net VCC
Other:
- board text added: "00-512kB 01-256kB 10-192kB 11-128kB"
- board text removed: "00-512kB 10-256kB 10-192kB 11-128kB"
- board text removed: "www.va-de-retro.com"
